File: board/MasTer_Controler_Route_Fix.brd (EAGLE design)
At the start: 118.1 x 96.2 mm, 58 parts, among them IC1 MEGA8535-P, IC2 DS1307, IC3 7805TV, P1 FSM, Q1 32,767kHz, Q10 IRF540, Q2 12MHz, Q3 BD139, Q4 IRF540, Q5 BD139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

Commit message: Board diedit
Connections:
- net N$20 renamed ADCMC
- net N$21 renamed ADCMD
- net N$26 renamed KATUP1
- net N$27 renamed KATUP2
- net N$29 renamed KATUP3
- net N$30 renamed KATUP4
- net N$32 renamed BUZZ
- net N$33 renamed MOTORD
- net N$34 renamed MOTORC
- net N$36 renamed FLOWS
Changed lines of the file:
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@@
 <?xml version="1.0" encoding="utf-8"?>
 <!DOCTYPE eagle SYSTEM "eagle.dtd">
-<eagle version="6.1">
+<eagle version="6.6.0">
 <drawing>
 <settings>
@@
 </class>
 </classes>
-<designrules>
+<designrules name="default">
 <description language="de">&lt;b&gt;EAGLE Design Rules&lt;/b&gt;
 &lt;p&gt;
@@
 <wire x1="86.36" y1="83.82" x2="86.36" y2="82.55" width="0.8128" layer="16"/>
 </signal>
-<signal name="N$20">
+<signal name="ADCMC">
 <contactref element="IC1" pad="33"/>
 <contactref element="JP2" pad="1"/>
 <wire x1="67.31" y1="60.96" x2="59.69" y2="60.96" width="0.8128" layer="16"/>
 </signal>
-<signal name="N$21">
+<signal name="ADCMD">
 <contactref element="JP2" pad="2"/>
 <contactref element="IC1" pad="34"/>
@@
 <wire x1="59.69" y1="73.66" x2="67.31" y2="73.66" width="0.8128" layer="16"/>
 </signal>
-<signal name="N$26">
+<signal name="KATUP1">
 <contactref element="IC1" pad="5"/>
 <contactref element="JP3" pad="1"/>
 <wire x1="38.1" y1="68.58" x2="44.45" y2="68.58" width="1.016" layer="16"/>
 </signal>
-<signal name="N$27">
+<signal name="KATUP2">
 <contactref element="JP3" pad="2"/>
 <contactref element="IC1" pad="4"/>
@@
 <wire x1="38.1" y1="73.66" x2="44.45" y2="73.66" width="1.016" layer="16"/>
 </signal>
-<signal name="N$29">
+<signal name="KATUP3">
 <contactref element="JP3" pad="4"/>
 <contactref element="IC1" pad="2"/>
 <wire x1="38.1" y1="76.2" x2="44.45" y2="76.2" width="1.016" layer="16"/>
 </signal>
-<signal name="N$30">
+<signal name="KATUP4">
 <contactref element="IC1" pad="1"/>
 <contactref element="JP3" pad="5"/>
@@
 <wire x1="57.15" y1="30.48" x2="59.69" y2="30.48" width="0.8128" layer="16"/>
 </signal>
-<signal name="N$32">
+<signal name="BUZZ">
 <contactref element="IC1" pad="20"/>
 <contactref element="JP4" pad="2"/>
 <wire x1="33.02" y1="30.48" x2="44.45" y2="30.48" width="0.8128" layer="16"/>
 </signal>
-<signal name="N$33">
+<signal name="MOTORD">
 <contactref element="IC1" pad="19"/>
 <contactref element="JP4" pad="3"/>
 <wire x1="44.45" y1="33.02" x2="33.02" y2="33.02" width="0.8128" layer="16"/>
 </signal>
-<signal name="N$34">
+<signal name="MOTORC">
 <contactref element="IC1" pad="18"/>
 <contactref element="JP4" pad="4"/>
@@
 <wire x1="44.45" y1="38.1" x2="33.02" y2="38.1" width="0.8128" layer="16"/>
 </signal>
-<signal name="N$36">
+<signal name="FLOWS">
 <contactref element="IC1" pad="16"/>
 <contactref element="JP4" pad="6"/>
